Commit message: modified camera position to belly

File: robbie/urdf/robbie.xacro (robot description, xacro)
@@ -136,5 +136,5 @@
     <parent link="chassis"/>
     <child link="camera_link"/>
-    <origin xyz="${chassis_length/2} 0 ${chassis_height/2+camera_height/2}"/>
+    <origin xyz="0 0 -${chassis_height/2 + camera_height/2}" rpy="0 1.5708 0"/>
   </joint>
   <gazebo reference="chassis">
@@ -171,9 +171,12 @@
     </plugin>
   </gazebo> -->
+  <gazebo reference="chassis">
+    <gravity>0</gravity>
+  </gazebo>
   <gazebo reference="camera_link">
     <sensor type="camera" name="camera1">
       <update_rate>30.0</update_rate>
       <camera name="head">
-        <horizontal_fov>1.3962634</horizontal_fov>
+        <horizontal_fov>1.5</horizontal_fov>
         <image>
           <width>800</width>
